File: hardware/pcbs/fmc_memory_adapter/fmc_memory_adapter.kicad_sch (KiCad schematic)
At the start: 38 parts, among them IC1 SN74AVC8T245PWG4, IC2 SN74AVC8T245PWG4, IC3 SN74AVC8T245PWG4, IC4 SN74AVC8T245PWG4, IC5 SN74AVC8T245PWG4, IC6 SN74AVC8T245PWG4, J1 GND_Jumper1, J10 Conn_02x08_Odd_Even, J2 GND_Jumper2, J3 GND_Jumper3, J4 GND_Jumper4, J5 GND_Jumper5, J7 Conn_02x03_Odd_Even, J8 ASP-134488-02, J9 Conn_01x03, P1 CONN_02X32_DISCO1_LEFT_BACK, P2 CONN_02X32_DISCO1_RIGHT_BACK

Commit message: Add PCI-E debugging interface connector to PCB
Parts:
- removed J4: GND_Jumper4, Connector_PinHeader_2.54mm:PinHeader_1x02_P2.54mm_Vertical, symbol Connector_Generic:Conn_02x01
- added J11: Conn_02x07_Odd_Even, Connector_PinHeader_2.54mm:PinHeader_2x07_P2.54mm_Vertical, symbol Connector_Generic:Conn_02x07_Odd_Even
- added J6: PCIE Breakout Adapter, custom_footprints:PCIE_1001878310010TLF, symbol pci_connector_custom:PCI_Connector_Custom
- J2: value GND_Jumper2 -> GND_Jumper3
Connections:
- net GND: now also J11.13 (Pin_13)
- net at J10.3 (Pin_3): now also J1.2 (Pin_2), J10.1 (Pin_1); no longer J2.2 (Pin_2)
- net at J3.2 (Pin_2): now also J10.7 (Pin_7); no longer J10.5 (Pin_5)
- net at J8.A1: now also J1.1 (Pin_1), J8.A4, J8.A5, J11.1 (Pin_1)
- net at J8.A12: now also J5.1 (Pin_1), J8.A13, J11.7 (Pin_7)
- net at J8.A16: now also J3.1 (Pin_1), J8.A17, J11.5 (Pin_5)
- net at J8.A8: now also J2.1 (Pin_1), J8.A9, J11.3 (Pin_3)
- net at J8.C26: now also IC2.3 (A1); no longer IC2.4 (A2)
- net at J8.C27: now also IC2.4 (A2); no longer IC2.3 (A1)
- net at J8.C30: now also J6.B4
- net at J8.C31: now also J6.B5
- net at J8.D31: now also J6.B7
- net at J8.D32: now also J6.B6
- net at J8.D6: now also J8.D7, J6.A10, J6.B11
- net at J8.E39: now also J7.1 (Pin_1)
- net at J8.F40: now also J6.B14
- net at J8.G2: now also J6.B16
- net at J8.G3: now also J6.B15
- net at J8.H11: now also J6.B13; no longer J7.1 (Pin_1)
- net at J8.H2: now also J6.B1
- net at J8.H29: now also J6.B12
- net at J8.H31: now also J6.B8
- net at J8.H32: now also J6.B9
- net at J8.H4: now also J6.B18
- net at J8.H5: now also J6.B17
- new net: J11.9 (Pin_9), J6.A3, J8.D35
- new net: J11.11 (Pin_11), J6.B2, J8.C34
- new net: J11.10 (Pin_10), J11.12 (Pin_12), J11.14 (Pin_14), J11.2 (Pin_2), J11.4 (Pin_4), J11.6 (Pin_6), J11.8 (Pin_8)
- new net: J10.5 (Pin_5), J2.2 (Pin_2)
- no-connect marks 429 -> 422

Commit message: Update PCB
Parts:
- removed J10: Conn_02x08_Odd_Even, Connector_PinHeader_2.54mm:PinHeader_2x08_P2.54mm_Vertical, symbol Connector_Generic:Conn_02x08_Odd_Even
- added J4: Conn_01x04_Pin, Connector_PinHeader_2.54mm:PinHeader_1x04_P2.54mm_Vertical, symbol Connector:Conn_01x04_Pin
- J6: value PCIE Breakout Adapter -> ~
Connections:
- net at C10.1, C12.1, C2.1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: now also J11.5 (Pin_5), J3.2 (Pin_2)
- net at C1.1, C11.1, C3.2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: now also J11.3 (Pin_3), J2.2 (Pin_2)
- net at J3.1 (Pin_1), J8.A16, J8.A17: no longer J11.5 (Pin_5)
- net at J6.B11, J8.D6, J8.D7: now also J6.B10; no longer J6.A10
- net at J11.9 (Pin_9), J8.D35: now also J6.B3; no longer J6.A3
- net at J1.1 (Pin_1), J8.A1, J8.A4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: no longer J11.1 (Pin_1)
- net at J2.1 (Pin_1), J8.A8, J8.A9: no longer J11.3 (Pin_3)
- net at J5.1 (Pin_1), J8.A12, J8.A13: no longer J11.7 (Pin_7)
- net at J5.2 (Pin_2): now also J11.7 (Pin_7), J4.1 (Pin_1), J4.2 (Pin_2), J4.3 (Pin_3), J4.4 (Pin_4)
- net at P1.30 (GND), P1.63 (GND), P1.64 (GND): now also J1.2 (Pin_2), J11.1 (Pin_1), P2.63 (GND), P2.64 (GND)
- no-connect marks 422 -> 418

Commit message: Improve grounding in pcb design
Parts:
- removed J2, J3: GND_Jumper3, Connector_PinHeader_2.54mm:PinHeader_1x02_P2.54mm_Vertical, symbol Connector_Generic:Conn_02x01
- removed J5: GND_Jumper5, Connector_PinHeader_2.54mm:PinHeader_1x02_P2.54mm_Vertical, symbol Connector_Generic:Conn_02x01
- removed J6: ~, custom_footprints:PCIE_1001878310010TLF, symbol pci_connector_custom:PCI_Connector_Custom
- added J2: PCI-E Extension/Debug Socket, custom_footprints:PCIE_1001878310010TLF, symbol pci_connector_custom:PCI_Connector_Custom
Connections:
- net GND: now also C1.1, C10.1, C11.1, C12.1, C2.1, C3.2, C4.2, C5.1, C6.1, C7.1, C8.1, C9.1, IC1.11 (GND_1), IC1.12 (GND_2), IC1.13 (GND_3), IC2.11 (GND_1), IC2.12 (GND_2), IC2.13 (GND_3), IC3.11 (GND_1), IC3.12 (GND_2), IC3.13 (GND_3), IC4.11 (GND_1), IC4.12 (GND_2), IC4.13 (GND_3), IC5.11 (GND_1), IC5.12 (GND_2), IC5.13 (GND_3), IC6.11 (GND_1), IC6.12 (GND_2), IC6.13 (GND_3), J11.10 (Pin_10), J11.12 (Pin_12), J11.14 (Pin_14), J11.2 (Pin_2), J11.4 (Pin_4), J11.6 (Pin_6), J11.8 (Pin_8); no longer J11.13 (Pin_13)
- net at J8.A16, J8.A17: now also J11.5 (Pin_5)
- net at J11.11 (Pin_11), J8.C34: now also J2.B2
- net at J11.7 (Pin_7), J4.1 (Pin_1), J4.2 (Pin_2)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: now also J8.A12, J8.A13
- net at J11.9 (Pin_9), J8.D35: now also J2.B3
- net at J8.A8, J8.A9: now also J11.3 (Pin_3)
- net at J8.C30: now also J2.B4
- net at J8.C31: now also J2.B5
- net at J8.D31: now also J2.B7
- net at J8.D32: now also J2.B6
- net at J8.D6, J8.D7: now also J2.B10, J2.B11
- net at J8.F40: now also J2.B14
- net at J8.G2: now also J2.B16
- net at J8.G3: now also J2.B15
- net at J8.H11: now also J2.B13
- net at J8.H2: now also J2.B1
- net at J8.H29: now also J2.B12
- net at J8.H31: now also J2.B8
- net at J8.H32: now also J2.B9
- net at J8.H4: now also J2.B18
- net at J8.H5: now also J2.B17
- no-connect marks 418 -> 419
Other:
- moved on the sheet: H1, H2, H3, H4, H5, H6, H7, H8, H9

Commit message: Update PCB
Connections:
- net GND: now also J11.5 (Pin_5), J8.A16, J8.A17
Changed lines of the file:
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@@
 	)
 	(junction
-		(at 186.69 284.48)
-		(diameter 0)
-		(color 0 0 0 0)
-	)
-	(junction
 		(at 177.8 162.56)
 		(diameter 0)
@@
 	)
 	(junction
+		(at 186.69 284.48)
+		(diameter 0)
+		(color 0 0 0 0)
+	)
+	(junction
 		(at 256.54 154.94)
 		(diameter 0)
@@
 	(wire
 		(pts
-			(xy 186.69 284.48) (xy 27.94 284.48)
-		)
-		(stroke
-			(width 0)
-			(type default)
-		)
-	)
-	(wire
-		(pts
 			(xy 119.38 90.17) (xy 137.16 90.17)
 		)
@@
 	(wire
 		(pts
-			(xy 27.94 284.48) (xy 27.94 91.44)
-		)
-		(stroke
-			(width 0)
-			(type default)
-		)
-	)
-	(wire
-		(pts
 			(xy 345.44 331.47) (xy 349.25 331.47)
 		)
@@
 		(length 2.54)
 		(shape round)
+		(at 33.02 91.44 0)
+		(fields_autoplaced yes)
+		(effects
+			(font
+				(size 1.27 1.27)
+			)
+			(justify left bottom)
+		)
+		(property "Netclass" "GND"
+			(at 33.7185 88.9 0)
+			(effects
+				(font
+					(size 1.27 1.27)
+					(italic yes)
+				)
+				(justify left)
+			)
+		)
+	)
+	(netclass_flag ""
+		(length 2.54)
+		(shape round)
 		(at 115.57 86.36 180)
 		(fields_autoplaced yes)
@@
 	(netclass_flag ""
 		(length 2.54)
+		(shape round)
+		(at 189.23 262.89 270)
+		(fields_autoplaced yes)
+		(effects
+			(font
+				(size 1.27 1.27)
+			)
+			(justify right bottom)
+		)
+		(property "Netclass" "GND"
+			(at 191.77 262.1915 90)
+			(effects
+				(font
+					(size 1.27 1.27)
+					(italic yes)
+				)
+				(justify left)
+			)
+		)
+	)
+	(netclass_flag ""
+		(length 2.54)
+		(shape round)
+		(at 179.07 260.35 270)
+		(fields_autoplaced yes)
+		(effects
+			(font
+				(size 1.27 1.27)
+			)
+			(justify right bottom)
+		)
+		(property "Netclass" "GND"
+			(at 181.61 259.6515 90)
+			(effects
+				(font
+					(size 1.27 1.27)
+					(italic yes)
+				)
+				(justify left)
+			)
+		)
+	)
+	(netclass_flag ""
+		(length 2.54)
 		(shape dot)
 		(at 175.26 110.49 0)
@@
 	)
 	(symbol
+		(lib_id "power:GND")
+		(at 186.69 284.48 0)
+		(unit 1)
+		(exclude_from_sim no)
+		(in_bom yes)
+		(on_board yes)
+		(dnp no)
+		(fields_autoplaced yes)
+		(property "Reference" "#PWR015"
+			(at 186.69 290.83 0)
+			(effects
+				(font
+					(size 1.27 1.27)
+				)
+				(hide yes)
+			)
+		)
+		(property "Value" "GND"
+			(at 186.69 289.56 0)
+			(effects
+				(font
+					(size 1.27 1.27)
+				)
+			)
+		)
+		(property "Footprint" ""
+			(at 186.69 284.48 0)
+			(effects
+				(font
+					(size 1.27 1.27)
+				)
+				(hide yes)
+			)
+		)
+		(property "Datasheet" ""
+			(at 186.69 284.48 0)
+			(effects
+				(font
+					(size 1.27 1.27)
+				)
+				(hide yes)
+			)
+		)
+		(property "Description" "Power symbol creates a global label with name \"GND\" , ground"
+			(at 186.69 284.48 0)
+			(effects
+				(font
+					(size 1.27 1.27)
+				)
+				(hide yes)
+			)
+		)
+		(pin "1"
+		)
+		(instances
+			(project ""
+				(path "/87c78429-be2b-40ed-8d3b-56cb9666a56f"
+					(reference "#PWR015")
+					(unit 1)
+				)
+			)
+		)
+	)
+	(symbol
 		(lib_id "C0805C104K5RAC7411:C0805C104K5RAC7411")
 		(at 321.31 128.27 0)
@@
 					(unit 1)
 				)
+			)
+		)
+	)
+	(symbol
+		(lib_id "power:GND")
+		(at 27.94 91.44 0)
+		(unit 1)
+		(exclude_from_sim no)
+		(in_bom yes)
+		(on_board yes)
+		(dnp no)
+		(fields_autoplaced yes)
+		(property "Reference" "#PWR013"
+			(at 27.94 97.79 0)
+			(effects
+				(font
+					(size 1.27 1.27)
+				)
+				(hide yes)
+			)
+		)
+		(property "Value" "GND"
+			(at 27.94 96.52 0)
+			(effects
+				(font
+					(size 1.27 1.27)
+				)
+			)
+		)
+		(property "Footprint" ""
+			(at 27.94 91.44 0)
+			(effects
+				(font
+					(size 1.27 1.27)
+				)
+				(hide yes)
+			)
+		)
+		(property "Datasheet" ""
+			(at 27.94 91.44 0)
+			(effects
+				(font
+					(size 1.27 1.27)
+				)
+				(hide yes)
+			)
+		)
+		(property "Description" "Power symbol creates a global label with name \"GND\" , ground"
+			(at 27.94 91.44 0)
+			(effects
+				(font
+					(size 1.27 1.27)
+				)
+				(hide yes)
+			)
+		)
+		(pin "1"
+		)
+		(instances
+			(project ""
+				(path "/87c78429-be2b-40ed-8d3b-56cb9666a56f"
+					(reference "#PWR013")
+					(unit 1)
+				)
