File: hardware/pcbs/fmc_memory_adapter/fmc_memory_adapter.kicad_sch (KiCad schematic)
At the start: 39 parts, among them IC1 SN74AVC8T245PWG4, IC2 SN74AVC8T245PWG4, IC3 SN74AVC8T245PWG4, IC4 SN74AVC8T245PWG4, IC5 SN74AVC8T245PWG4, IC6 SN74AVC8T245PWG4, J1 GND_Jumper1, J11 Conn_02x07_Odd_Even, J2 GND_Jumper3, J3 GND_Jumper3, J4 Conn_01x04_Pin, J5 GND_Jumper5, J7 Conn_02x03_Odd_Even, J8 ASP-134488-02, J9 Conn_01x03, P1 CONN_02X32_DISCO1_LEFT_BACK, P2 CONN_02X32_DISCO1_RIGHT_BACK

Commit message: Update README for ps firmware
Parts:
- removed J2, J3: GND_Jumper3, Connector_PinHeader_2.54mm:PinHeader_1x02_P2.54mm_Vertical, symbol Connector_Generic:Conn_02x01
- removed J5: GND_Jumper5, Connector_PinHeader_2.54mm:PinHeader_1x02_P2.54mm_Vertical, symbol Connector_Generic:Conn_02x01
- removed J6: ~, custom_footprints:PCIE_1001878310010TLF, symbol pci_connector_custom:PCI_Connector_Custom
- added J2: PCI-E Extension/Debug Socket, custom_footprints:PCIE_1001878310010TLF, symbol pci_connector_custom:PCI_Connector_Custom
Connections:
- net GND: now also C1.1, C10.1, C11.1, C12.1, C2.1, C3.2, C4.2, C5.1, C6.1, C7.1, C8.1, C9.1, IC1.11 (GND_1), IC1.12 (GND_2), IC1.13 (GND_3), IC2.11 (GND_1), IC2.12 (GND_2), IC2.13 (GND_3), IC3.11 (GND_1), IC3.12 (GND_2), IC3.13 (GND_3), IC4.11 (GND_1), IC4.12 (GND_2), IC4.13 (GND_3), IC5.11 (GND_1), IC5.12 (GND_2), IC5.13 (GND_3), IC6.11 (GND_1), IC6.12 (GND_2), IC6.13 (GND_3), J11.10 (Pin_10), J11.12 (Pin_12), J11.14 (Pin_14), J11.2 (Pin_2), J11.4 (Pin_4), J11.5 (Pin_5), J11.6 (Pin_6), J11.7 (Pin_7), J11.8 (Pin_8), J4.1 (Pin_1), J4.2 (Pin_2), J4.3 (Pin_3), J4.4 (Pin_4), J8.A12, J8.A13, J8.A16, J8.A17; no longer J11.13 (Pin_13)
- net at J11.11 (Pin_11), J8.C34: now also J2.B2
- net at J11.9 (Pin_9), J8.D35: now also J2.B3
- net at J8.A8, J8.A9: now also J11.3 (Pin_3)
- net at J8.C30: now also J2.B4
- net at J8.C31: now also J2.B5
- net at J8.D31: now also J2.B7
- net at J8.D32: now also J2.B6
- net at J8.D6, J8.D7: now also J2.B10, J2.B11
- net at J8.F40: now also J2.B14
- net at J8.G2: now also J2.B16
- net at J8.G3: now also J2.B15
- net at J8.H11: now also J2.B13
- net at J8.H2: now also J2.B1
- net at J8.H29: now also J2.B12
- net at J8.H31: now also J2.B8
- net at J8.H32: now also J2.B9
- net at J8.H4: now also J2.B18
- net at J8.H5: now also J2.B17
- no-connect marks 418 -> 419
Other:
- moved on the sheet: H1, H2, H3, H4, H5, H6, H7, H8, H9
